File: hardware/SB_interface/SB_interface.kicad_pcb (KiCad board)
At the start: 2 copper layers, 147.4 x 208.5 mm, 231 parts, among them J1 8P8C_TelPairs, J2 8P8C_TelPairs, J3 8P8C_TelPairs, J4 Conn_01x09_Pin, J5 Screw_Terminal_01x02, J6 Screw_Terminal_01x02, J7 EXTENSION HDR., J8 Jack-DC, K1 J104D2C12VDC.36S, K10 J104D2C12VDC.36S, K11 J104D2C12VDC.36S, K12 J104D2C12VDC.36S, K13 J104D2C12VDC.36S, K2 J104D2C12VDC.36S, K3 J104D2C12VDC.36S, K4 J104D2C12VDC.36S, K5 J104D2C12VDC.36S, K6 J104D2C12VDC.36S, K7 J104D2C12VDC.36S, K8 J104D2C12VDC.36S, K9 J104D2C12VDC.36S, Q1 2N7002, Q10 2N7002, Q11 MMBTA42, Q12 MMBTA42, Q13 2N7002, Q14 MMBTA42, Q15 MMBTA42, Q16 2N7002, Q17 MMBTA42, Q18 MMBTA42, Q19 2N7002, Q2 MMBTA42, Q20 MMBTA42, Q21 MMBTA42, Q22 2N7002, Q23 MMBTA42, Q24 MMBTA42, Q25 2N7002, Q26 MMBTA42, Q27 MMBTA42, Q28 2N7002, Q29 MMBTA42, Q3 MMBTA42, Q30 MMBTA42, Q31 2N7002, Q32 MMBTA42, Q33 MMBTA42, Q34 2N7002, Q35 MMBTA42, Q36 MMBTA42, Q37 2N7002, Q4 2N7002, Q5 MMBTA42, Q6 MMBTA42, Q7 2N7002, Q8 MMBTA42, Q9 MMBTA42, U1 MCP23017_SP, U2 MCP23017_SP

Commit message: added prototyping area
Parts:
- added J9: EXTENSION HDR., Connector_PinHeader_2.54mm:PinHeader_1x07_P2.54mm_Vertical, F.Cu at (160.3, 187.5)
- added REF**: breadboard_pin, sb_interface:breadboard_pin, F.Cu at (144.8, 119.4)
- added REF**: breadboard_pin, sb_interface:breadboard_pin, F.Cu at (139.7, 147.3)
- added REF**: breadboard_pin, sb_interface:breadboard_pin, F.Cu at (162.6, 144.8)
- added REF**: breadboard_pin, sb_interface:breadboard_pin, F.Cu at (167.6, 134.6)
- added REF**: breadboard_pin, sb_interface:breadboard_pin, F.Cu at (149.9, 119.4)
- added REF**: breadboard_pin, sb_interface:breadboard_pin, F.Cu at (162.6, 99.1)
- added REF**: breadboard_pin, sb_interface:breadboard_pin, F.Cu at (172.7, 144.8)
- added REF**: breadboard_pin, sb_interface:breadboard_pin, F.Cu at (157.5, 83.8)
- added REF**: breadboard_pin, sb_interface:breadboard_pin, F.Cu at (139.7, 149.9)
- added REF**: breadboard_pin, sb_interface:breadboard_pin, F.Cu at (142.2, 104.1)
- added REF**: breadboard_pin, sb_interface:breadboard_pin, F.Cu at (147.3, 114.3)
- added REF**: BLABLAPIN, sb_interface:breadboard_pin, F.Cu at (172.7, 165.1)
- added REF**: breadboard_pin, sb_interface:breadboard_pin, F.Cu at (157.5, 109.2)
- added REF**: breadboard_pin, sb_interface:breadboard_pin, F.Cu at (142.2, 119.4)
- added REF**: breadboard_pin, sb_interface:breadboard_pin, F.Cu at (172.7, 116.8)
- added REF**: breadboard_pin, sb_interface:breadboard_pin, F.Cu at (149.9, 106.7)
- added REF**: breadboard_pin, sb_interface:breadboard_pin, F.Cu at (157.5, 152.4)
- added REF**: breadboard_pin, sb_interface:breadboard_pin, F.Cu at (144.8, 147.3)
- added REF**: breadboard_pin, sb_interface:breadboard_pin, F.Cu at (154.9, 76.2)
- added REF**: breadboard_pin, sb_interface:breadboard_pin, F.Cu at (152.4, 83.8)
- added REF**: breadboard_pin, sb_interface:breadboard_pin, F.Cu at (160.0, 121.9)
- added REF**: breadboard_pin, sb_interface:breadboard_pin, F.Cu at (160.0, 147.3)
- added REF**: breadboard_pin, sb_interface:breadboard_pin, F.Cu at (134.6, 78.7)
- added REF**: breadboard_pin, sb_interface:breadboard_pin, F.Cu at (137.2, 76.2)
- added REF**: breadboard_pin, sb_interface:breadboard_pin, F.Cu at (142.2, 134.6)
- added REF**: breadboard_pin, sb_interface:breadboard_pin, F.Cu at (142.2, 78.7)
- added REF**: breadboard_pin, sb_interface:breadboard_pin, F.Cu at (137.2, 104.1)
- added REF**: breadboard_pin, sb_interface:breadboard_pin, F.Cu at (137.2, 127.0)
- added REF**: breadboard_pin, sb_interface:breadboard_pin, F.Cu at (137.2, 152.4)
- added REF**: breadboard_pin, sb_interface:breadboard_pin, F.Cu at (167.6, 73.7)
- added REF**: breadboard_pin, sb_interface:breadboard_pin, F.Cu at (144.8, 73.7)
- added REF**: breadboard_pin, sb_interface:breadboard_pin, F.Cu at (142.2, 121.9)
- added REF**: breadboard_pin, sb_interface:breadboard_pin, F.Cu at (134.6, 104.1)
- added REF**: breadboard_pin, sb_interface:breadboard_pin, F.Cu at (162.6, 134.6)
- added REF**: breadboard_pin, sb_interface:breadboard_pin, F.Cu at (134.6, 132.1)
- added REF**: breadboard_pin, sb_interface:breadboard_pin, F.Cu at (147.3, 129.5)
- added REF**: breadboard_pin, sb_interface:breadboard_pin, F.Cu at (172.7, 129.5)
- added REF**: breadboard_pin, sb_interface:breadboard_pin, F.Cu at (170.2, 152.4)
- added REF**: breadboard_pin, sb_interface:breadboard_pin, F.Cu at (154.9, 121.9)
- added REF**: breadboard_pin, sb_interface:breadboard_pin, F.Cu at (154.9, 124.5)
- added REF**: breadboard_pin, sb_interface:breadboard_pin, F.Cu at (167.6, 114.3)
- added REF**: breadboard_pin, sb_interface:breadboard_pin, F.Cu at (162.6, 88.9)
- added REF**: breadboard_pin, sb_interface:breadboard_pin, F.Cu at (134.6, 139.7)
- added REF**: breadboard_pin, sb_interface:breadboard_pin, F.Cu at (144.8, 132.1)
- added REF**: breadboard_pin, sb_interface:breadboard_pin, F.Cu at (160.0, 144.8)
- added REF**: breadboard_pin, sb_interface:breadboard_pin, F.Cu at (139.7, 160.0)
- added REF**: breadboard_pin, sb_interface:breadboard_pin, F.Cu at (154.9, 142.2)
- added REF**: breadboard_pin, sb_interface:breadboard_pin, F.Cu at (170.2, 94.0)
- added REF**: breadboard_pin, sb_interface:breadboard_pin, F.Cu at (149.9, 152.4)
- added REF**: breadboard_pin, sb_interface:breadboard_pin, F.Cu at (172.7, 96.5)
- added REF**: breadboard_pin, sb_interface:breadboard_pin, F.Cu at (139.7, 119.4)
- added REF**: breadboard_pin, sb_interface:breadboard_pin, F.Cu at (149.9, 83.8)
- added REF**: breadboard_pin, sb_interface:breadboard_pin, F.Cu at (147.3, 109.2)
- added REF**: breadboard_pin, sb_interface:breadboard_pin, F.Cu at (144.8, 152.4)
- added REF**: breadboard_pin, sb_interface:breadboard_pin, F.Cu at (134.6, 83.8)
- added REF**: breadboard_pin, sb_interface:breadboard_pin, F.Cu at (154.9, 114.3)
- added REF**: breadboard_pin, sb_interface:breadboard_pin, F.Cu at (165.1, 149.9)
- added REF**: breadboard_pin, sb_interface:breadboard_pin, F.Cu at (149.9, 109.2)
- added REF**: breadboard_pin, sb_interface:breadboard_pin, F.Cu at (147.3, 139.7)
- added REF**: breadboard_pin, sb_interface:breadboard_pin, F.Cu at (134.6, 106.7)
- added REF**: breadboard_pin, sb_interface:breadboard_pin, F.Cu at (157.5, 88.9)
- added REF**: breadboard_pin, sb_interface:breadboard_pin, F.Cu at (142.2, 142.2)
- added REF**: breadboard_pin, sb_interface:breadboard_pin, F.Cu at (137.2, 116.8)
- added REF**: breadboard_pin, sb_interface:breadboard_pin, F.Cu at (154.9, 109.2)
- added REF**: breadboard_pin, sb_interface:breadboard_pin, F.Cu at (154.9, 165.1)
- added REF**: breadboard_pin, sb_interface:breadboard_pin, F.Cu at (160.0, 106.7)
- added REF**: breadboard_pin, sb_interface:breadboard_pin, F.Cu at (147.3, 157.5)
- added REF**: breadboard_pin, sb_interface:breadboard_pin, F.Cu at (165.1, 94.0)
- added REF**: breadboard_pin, sb_interface:breadboard_pin, F.Cu at (172.7, 149.9)
- added REF**: breadboard_pin, sb_interface:breadboard_pin, F.Cu at (152.4, 152.4)
- added REF**: breadboard_pin, sb_interface:breadboard_pin, F.Cu at (142.2, 114.3)
- added REF**: breadboard_pin, sb_interface:breadboard_pin, F.Cu at (139.7, 68.6)
- added REF**: breadboard_pin, sb_interface:breadboard_pin, F.Cu at (134.6, 109.2)
- added REF**: breadboard_pin, sb_interface:breadboard_pin, F.Cu at (154.9, 73.7)
- added REF**: breadboard_pin, sb_interface:breadboard_pin, F.Cu at (172.7, 127.0)
- added REF**: breadboard_pin, sb_interface:breadboard_pin, F.Cu at (147.3, 104.1)
- added REF**: breadboard_pin, sb_interface:breadboard_pin, F.Cu at (157.5, 78.7)
- added REF**: breadboard_pin, sb_interface:breadboard_pin, F.Cu at (165.1, 91.4)
- added REF**: breadboard_pin, sb_interface:breadboard_pin, F.Cu at (144.8, 129.5)
- added REF**: breadboard_pin, sb_interface:breadboard_pin, F.Cu at (165.1, 116.8)
- added REF**: breadboard_pin, sb_interface:breadboard_pin, F.Cu at (170.2, 114.3)
- added REF**: breadboard_pin, sb_interface:breadboard_pin, F.Cu at (139.7, 114.3)
- added REF**: breadboard_pin, sb_interface:breadboard_pin, F.Cu at (172.7, 132.1)
- added REF**: breadboard_pin, sb_interface:breadboard_pin, F.Cu at (172.7, 147.3)
- added REF**: breadboard_pin, sb_interface:breadboard_pin, F.Cu at (167.6, 160.0)
- added REF**: breadboard_pin, sb_interface:breadboard_pin, F.Cu at (142.2, 109.2)
- added REF**: breadboard_pin, sb_interface:breadboard_pin, F.Cu at (139.7, 144.8)
- added REF**: breadboard_pin, sb_interface:breadboard_pin, F.Cu at (160.0, 111.8)
- added REF**: breadboard_pin, sb_interface:breadboard_pin, F.Cu at (167.6, 144.8)
- added REF**: breadboard_pin, sb_interface:breadboard_pin, F.Cu at (160.0, 73.7)
- added REF**: breadboard_pin, sb_interface:breadboard_pin, F.Cu at (134.6, 73.7)
- added REF**: breadboard_pin, sb_interface:breadboard_pin, F.Cu at (137.2, 129.5)
- added REF**: breadboard_pin, sb_interface:breadboard_pin, F.Cu at (134.6, 152.4)
- added REF**: breadboard_pin, sb_interface:breadboard_pin, F.Cu at (147.3, 73.7)
- added REF**: breadboard_pin, sb_interface:breadboard_pin, F.Cu at (147.3, 149.9)
- added REF**: breadboard_pin, sb_interface:breadboard_pin, F.Cu at (144.8, 154.9)
- added REF**: breadboard_pin, sb_interface:breadboard_pin, F.Cu at (154.9, 83.8)
- added REF**: breadboard_pin, sb_interface:breadboard_pin, F.Cu at (149.9, 78.7)
- added REF**: breadboard_pin, sb_interface:breadboard_pin, F.Cu at (157.5, 139.7)
- added REF**: breadboard_pin, sb_interface:breadboard_pin, F.Cu at (149.9, 104.1)
- added REF**: breadboard_pin, sb_interface:breadboard_pin, F.Cu at (134.6, 116.8)
- added REF**: breadboard_pin, sb_interface:breadboard_pin, F.Cu at (162.6, 139.7)
- added REF**: breadboard_pin, sb_interface:breadboard_pin, F.Cu at (144.8, 121.9)
- added REF**: breadboard_pin, sb_interface:breadboard_pin, F.Cu at (160.0, 119.4)
- added REF**: breadboard_pin, sb_interface:breadboard_pin, F.Cu at (157.5, 147.3)
- added REF**: breadboard_pin, sb_interface:breadboard_pin, F.Cu at (157.5, 137.2)
- added REF**: breadboard_pin, sb_interface:breadboard_pin, F.Cu at (152.4, 91.4)
- added REF**: breadboard_pin, sb_interface:breadboard_pin, F.Cu at (165.1, 83.8)
- added REF**: breadboard_pin, sb_interface:breadboard_pin, F.Cu at (139.7, 139.7)
- added REF**: breadboard_pin, sb_interface:breadboard_pin, F.Cu at (147.3, 76.2)
- added REF**: breadboard_pin, sb_interface:breadboard_pin, F.Cu at (162.6, 96.5)
- added REF**: breadboard_pin, sb_interface:breadboard_pin, F.Cu at (147.3, 111.8)
- added REF**: breadboard_pin, sb_interface:breadboard_pin, F.Cu at (144.8, 139.7)
- added REF**: breadboard_pin, sb_interface:breadboard_pin, F.Cu at (144.8, 127.0)
- added REF**: breadboard_pin, sb_interface:breadboard_pin, F.Cu at (172.7, 88.9)
- added REF**: breadboard_pin, sb_interface:breadboard_pin, F.Cu at (152.4, 101.6)
- added REF**: breadboard_pin, sb_interface:breadboard_pin, F.Cu at (134.6, 68.6)
- added REF**: breadboard_pin, sb_interface:breadboard_pin, F.Cu at (172.7, 104.1)
- added REF**: breadboard_pin, sb_interface:breadboard_pin, F.Cu at (165.1, 121.9)
- added REF**: breadboard_pin, sb_interface:breadboard_pin, F.Cu at (160.0, 109.2)
- added REF**: breadboard_pin, sb_interface:breadboard_pin, F.Cu at (167.6, 94.0)
- added REF**: breadboard_pin, sb_interface:breadboard_pin, F.Cu at (134.6, 142.2)
- added REF**: breadboard_pin, sb_interface:breadboard_pin, F.Cu at (137.2, 119.4)
- added REF**: breadboard_pin, sb_interface:breadboard_pin, F.Cu at (157.5, 144.8)
- added REF**: breadboard_pin, sb_interface:breadboard_pin, F.Cu at (137.2, 149.9)
- added REF**: breadboard_pin, sb_interface:breadboard_pin, F.Cu at (167.6, 81.3)
- added REF**: breadboard_pin, sb_interface:breadboard_pin, F.Cu at (157.5, 127.0)
- added REF**: breadboard_pin, sb_interface:breadboard_pin, F.Cu at (137.2, 124.5)
- added REF**: breadboard_pin, sb_interface:breadboard_pin, F.Cu at (134.6, 91.4)
- added REF**: breadboard_pin, sb_interface:breadboard_pin, F.Cu at (149.9, 86.4)
- added REF**: breadboard_pin, sb_interface:breadboard_pin, F.Cu at (167.6, 68.6)
- added REF**: breadboard_pin, sb_interface:breadboard_pin, F.Cu at (142.2, 149.9)
- added REF**: breadboard_pin, sb_interface:breadboard_pin, F.Cu at (139.7, 154.9)
- added REF**: breadboard_pin, sb_interface:breadboard_pin, F.Cu at (137.2, 142.2)
- added REF**: breadboard_pin, sb_interface:breadboard_pin, F.Cu at (165.1, 119.4)
- added REF**: breadboard_pin, sb_interface:breadboard_pin, F.Cu at (160.0, 129.5)
- added REF**: breadboard_pin, sb_interface:breadboard_pin, F.Cu at (165.1, 147.3)
- added REF**: breadboard_pin, sb_interface:breadboard_pin, F.Cu at (162.6, 81.3)
- added REF**: breadboard_pin, sb_interface:breadboard_pin, F.Cu at (160.0, 68.6)
- added REF**: breadboard_pin, sb_interface:breadboard_pin, F.Cu at (137.2, 137.2)
- added REF**: breadboard_pin, sb_interface:breadboard_pin, F.Cu at (149.9, 147.3)
- added REF**: breadboard_pin, sb_interface:breadboard_pin, F.Cu at (172.7, 109.2)
- added REF**: breadboard_pin, sb_interface:breadboard_pin, F.Cu at (144.8, 78.7)
- added REF**: breadboard_pin, sb_interface:breadboard_pin, F.Cu at (139.7, 157.5)
- added REF**: breadboard_pin, sb_interface:breadboard_pin, F.Cu at (149.9, 88.9)
- added REF**: breadboard_pin, sb_interface:breadboard_pin, F.Cu at (147.3, 152.4)
- added REF**: breadboard_pin, sb_interface:breadboard_pin, F.Cu at (137.2, 134.6)
- added REF**: breadboard_pin, sb_interface:breadboard_pin, F.Cu at (160.0, 99.1)
- added REF**: breadboard_pin, sb_interface:breadboard_pin, F.Cu at (162.6, 137.2)
- added REF**: breadboard_pin, sb_interface:breadboard_pin, F.Cu at (147.3, 81.3)
- added REF**: breadboard_pin, sb_interface:breadboard_pin, F.Cu at (165.1, 154.9)
- added REF**: breadboard_pin, sb_interface:breadboard_pin, F.Cu at (139.7, 127.0)
- added REF**: breadboard_pin, sb_interface:breadboard_pin, F.Cu at (172.7, 86.4)
- added REF**: breadboard_pin, sb_interface:breadboard_pin, F.Cu at (137.2, 94.0)
- added REF**: breadboard_pin, sb_interface:breadboard_pin, F.Cu at (139.7, 111.8)
- added REF**: breadboard_pin, sb_interface:breadboard_pin, F.Cu at (154.9, 81.3)
- added REF**: breadboard_pin, sb_interface:breadboard_pin, F.Cu at (142.2, 86.4)
- added REF**: breadboard_pin, sb_interface:breadboard_pin, F.Cu at (139.7, 106.7)
- added REF**: breadboard_pin, sb_interface:breadboard_pin, F.Cu at (172.7, 78.7)
- added REF**: breadboard_pin, sb_interface:breadboard_pin, F.Cu at (162.6, 101.6)
- added REF**: breadboard_pin, sb_interface:breadboard_pin, F.Cu at (154.9, 134.6)
- added REF**: breadboard_pin, sb_interface:breadboard_pin, F.Cu at (170.2, 111.8)
- added REF**: breadboard_pin, sb_interface:breadboard_pin, F.Cu at (142.2, 116.8)
- added REF**: breadboard_pin, sb_interface:breadboard_pin, F.Cu at (134.6, 124.5)
- added REF**: breadboard_pin, sb_interface:breadboard_pin, F.Cu at (152.4, 114.3)
- added REF**: breadboard_pin, sb_interface:breadboard_pin, F.Cu at (160.0, 165.1)
- added REF**: breadboard_pin, sb_interface:breadboard_pin, F.Cu at (160.0, 154.9)
- added REF**: breadboard_pin, sb_interface:breadboard_pin, F.Cu at (170.2, 127.0)
- added REF**: breadboard_pin, sb_interface:breadboard_pin, F.Cu at (165.1, 73.7)
- added REF**: breadboard_pin, sb_interface:breadboard_pin, F.Cu at (134.6, 129.5)
- added REF**: breadboard_pin, sb_interface:breadboard_pin, F.Cu at (152.4, 124.5)
- added REF**: breadboard_pin, sb_interface:breadboard_pin, F.Cu at (160.0, 134.6)
- added REF**: breadboard_pin, sb_interface:breadboard_pin, F.Cu at (142.2, 139.7)
- added REF**: breadboard_pin, sb_interface:breadboard_pin, F.Cu at (137.2, 147.3)
- added REF**: breadboard_pin, sb_interface:breadboard_pin, F.Cu at (152.4, 88.9)
- added REF**: breadboard_pin, sb_interface:breadboard_pin, F.Cu at (167.6, 78.7)
- added REF**: breadboard_pin, sb_interface:breadboard_pin, F.Cu at (142.2, 152.4)
- added REF**: breadboard_pin, sb_interface:breadboard_pin, F.Cu at (147.3, 101.6)
- added REF**: breadboard_pin, sb_interface:breadboard_pin, F.Cu at (162.6, 83.8)
- added REF**: breadboard_pin, sb_interface:breadboard_pin, F.Cu at (144.8, 149.9)
- added REF**: breadboard_pin, sb_interface:breadboard_pin, F.Cu at (134.6, 147.3)
- added REF**: breadboard_pin, sb_interface:breadboard_pin, F.Cu at (154.9, 119.4)
- added REF**: breadboard_pin, sb_interface:breadboard_pin, F.Cu at (149.9, 154.9)
- added REF**: breadboard_pin, sb_interface:breadboard_pin, F.Cu at (142.2, 101.6)
- added REF**: breadboard_pin, sb_interface:breadboard_pin, F.Cu at (170.2, 109.2)
- added REF**: breadboard_pin, sb_interface:breadboard_pin, F.Cu at (154.9, 116.8)
- added REF**: breadboard_pin, sb_interface:breadboard_pin, F.Cu at (152.4, 149.9)
- added REF**: breadboard_pin, sb_interface:breadboard_pin, F.Cu at (154.9, 129.5)
- added REF**: breadboard_pin, sb_interface:breadboard_pin, F.Cu at (139.7, 73.7)
- added REF**: breadboard_pin, sb_interface:breadboard_pin, F.Cu at (165.1, 109.2)
- added REF**: breadboard_pin, sb_interface:breadboard_pin, F.Cu at (134.6, 127.0)
- added REF**: breadboard_pin, sb_interface:breadboard_pin, F.Cu at (157.5, 101.6)
- added REF**: breadboard_pin, sb_interface:breadboard_pin, F.Cu at (139.7, 124.5)
- added REF**: breadboard_pin, sb_interface:breadboard_pin, F.Cu at (152.4, 109.2)
- added REF**: breadboard_pin, sb_interface:breadboard_pin, F.Cu at (154.9, 106.7)
- added REF**: breadboard_pin, sb_interface:breadboard_pin, F.Cu at (139.7, 76.2)
- added REF**: breadboard_pin, sb_interface:breadboard_pin, F.Cu at (144.8, 81.3)
- added REF**: breadboard_pin, sb_interface:breadboard_pin, F.Cu at (142.2, 144.8)
- added REF**: breadboard_pin, sb_interface:breadboard_pin, F.Cu at (142.2, 106.7)
- added REF**: breadboard_pin, sb_interface:breadboard_pin, F.Cu at (170.2, 68.6)
- added REF**: breadboard_pin, sb_interface:breadboard_pin, F.Cu at (157.5, 154.9)
- added REF**: breadboard_pin, sb_interface:breadboard_pin, F.Cu at (139.7, 142.2)
- added REF**: breadboard_pin, sb_interface:breadboard_pin, F.Cu at (147.3, 119.4)
- added REF**: breadboard_pin, sb_interface:breadboard_pin, F.Cu at (137.2, 86.4)
- added REF**: breadboard_pin, sb_interface:breadboard_pin, F.Cu at (152.4, 127.0)
- added REF**: breadboard_pin, sb_interface:breadboard_pin, F.Cu at (144.8, 104.1)
- added REF**: breadboard_pin, sb_interface:breadboard_pin, F.Cu at (162.6, 142.2)
- added REF**: breadboard_pin, sb_interface:breadboard_pin, F.Cu at (152.4, 129.5)
- added REF**: breadboard_pin, sb_interface:breadboard_pin, F.Cu at (154.9, 88.9)
- added REF**: breadboard_pin, sb_interface:breadboard_pin, F.Cu at (170.2, 121.9)
- added REF**: breadboard_pin, sb_interface:breadboard_pin, F.Cu at (165.1, 139.7)
- added REF**: breadboard_pin, sb_interface:breadboard_pin, F.Cu at (167.6, 109.2)
- added REF**: breadboard_pin, sb_interface:breadboard_pin, F.Cu at (149.9, 157.5)
- added REF**: breadboard_pin, sb_interface:breadboard_pin, F.Cu at (160.0, 104.1)
- added REF**: breadboard_pin, sb_interface:breadboard_pin, F.Cu at (144.8, 157.5)
- added REF**: breadboard_pin, sb_interface:breadboard_pin, F.Cu at (139.7, 99.1)
- added REF**: breadboard_pin, sb_interface:breadboard_pin, F.Cu at (167.6, 83.8)
- added REF**: breadboard_pin, sb_interface:breadboard_pin, F.Cu at (170.2, 104.1)
- added REF**: breadboard_pin, sb_interface:breadboard_pin, F.Cu at (149.9, 127.0)
- added REF**: breadboard_pin, sb_interface:breadboard_pin, F.Cu at (154.9, 132.1)
- added REF**: breadboard_pin, sb_interface:breadboard_pin, F.Cu at (137.2, 121.9)
- added REF**: breadboard_pin, sb_interface:breadboard_pin, F.Cu at (160.0, 78.7)
- added REF**: breadboard_pin, sb_interface:breadboard_pin, F.Cu at (165.1, 99.1)
- added REF**: breadboard_pin, sb_interface:breadboard_pin, F.Cu at (172.7, 101.6)
- added REF**: breadboard_pin, sb_interface:breadboard_pin, F.Cu at (165.1, 132.1)
- added REF**: breadboard_pin, sb_interface:breadboard_pin, F.Cu at (137.2, 81.3)
- added REF**: breadboard_pin, sb_interface:breadboard_pin, F.Cu at (165.1, 142.2)
- added REF**: breadboard_pin, sb_interface:breadboard_pin, F.Cu at (147.3, 106.7)
- added REF**: breadboard_pin, sb_interface:breadboard_pin, F.Cu at (149.9, 160.0)
- added REF**: breadboard_pin, sb_interface:breadboard_pin, F.Cu at (172.7, 99.1)
- added REF**: breadboard_pin, sb_interface:breadboard_pin, F.Cu at (165.1, 134.6)
- added REF**: breadboard_pin, sb_interface:breadboard_pin, F.Cu at (167.6, 86.4)
- added REF**: breadboard_pin, sb_interface:breadboard_pin, F.Cu at (152.4, 104.1)
- added REF**: breadboard_pin, sb_interface:breadboard_pin, F.Cu at (139.7, 104.1)
- added REF**: breadboard_pin, sb_interface:breadboard_pin, F.Cu at (142.2, 94.0)
- added REF**: breadboard_pin, sb_interface:breadboard_pin, F.Cu at (165.1, 165.1)
- added REF**: breadboard_pin, sb_interface:breadboard_pin, F.Cu at (172.7, 124.5)
- added REF**: breadboard_pin, sb_interface:breadboard_pin, F.Cu at (139.7, 91.4)
- added REF**: breadboard_pin, sb_interface:breadboard_pin, F.Cu at (154.9, 139.7)
- added REF**: breadboard_pin, sb_interface:breadboard_pin, F.Cu at (149.9, 99.1)
- added REF**: breadboard_pin, sb_interface:breadboard_pin, F.Cu at (160.0, 83.8)
- added REF**: breadboard_pin, sb_interface:breadboard_pin, F.Cu at (134.6, 94.0)
- added REF**: breadboard_pin, sb_interface:breadboard_pin, F.Cu at (165.1, 104.1)
- added REF**: breadboard_pin, sb_interface:breadboard_pin, F.Cu at (167.6, 104.1)
- added REF**: breadboard_pin, sb_interface:breadboard_pin, F.Cu at (165.1, 78.7)
- added REF**: breadboard_pin, sb_interface:breadboard_pin, F.Cu at (137.2, 99.1)
- added REF**: breadboard_pin, sb_interface:breadboard_pin, F.Cu at (162.6, 152.4)
- added REF**: breadboard_pin, sb_interface:breadboard_pin, F.Cu at (165.1, 76.2)
- added REF**: breadboard_pin, sb_interface:breadboard_pin, F.Cu at (142.2, 132.1)
- added REF**: breadboard_pin, sb_interface:breadboard_pin, F.Cu at (142.2, 99.1)
- added REF**: breadboard_pin, sb_interface:breadboard_pin, F.Cu at (144.8, 160.0)
- added REF**: breadboard_pin, sb_interface:breadboard_pin, F.Cu at (157.5, 132.1)
- added REF**: breadboard_pin, sb_interface:breadboard_pin, F.Cu at (152.4, 68.6)
- added REF**: breadboard_pin, sb_interface:breadboard_pin, F.Cu at (170.2, 119.4)
- added REF**: breadboard_pin, sb_interface:breadboard_pin, F.Cu at (149.9, 132.1)
- added REF**: breadboard_pin, sb_interface:breadboard_pin, F.Cu at (134.6, 134.6)
- added REF**: breadboard_pin, sb_interface:breadboard_pin, F.Cu at (154.9, 99.1)
- added REF**: breadboard_pin, sb_interface:breadboard_pin, F.Cu at (162.6, 116.8)
- added REF**: breadboard_pin, sb_interface:breadboard_pin, F.Cu at (160.0, 91.4)
- added REF**: breadboard_pin, sb_interface:breadboard_pin, F.Cu at (157.5, 94.0)
- added REF**: breadboard_pin, sb_interface:breadboard_pin, F.Cu at (162.6, 73.7)
- added REF**: breadboard_pin, sb_interface:breadboard_pin, F.Cu at (144.8, 99.1)
- added REF**: breadboard_pin, sb_interface:breadboard_pin, F.Cu at (149.9, 139.7)
- added REF**: breadboard_pin, sb_interface:breadboard_pin, F.Cu at (137.2, 139.7)
- added REF**: breadboard_pin, sb_interface:breadboard_pin, F.Cu at (154.9, 68.6)
- added REF**: breadboard_pin, sb_interface:breadboard_pin, F.Cu at (170.2, 73.7)
- added REF**: breadboard_pin, sb_interface:breadboard_pin, F.Cu at (170.2, 116.8)
- added REF**: breadboard_pin, sb_interface:breadboard_pin, F.Cu at (142.2, 96.5)
- added REF**: breadboard_pin, sb_interface:breadboard_pin, F.Cu at (165.1, 114.3)
- added REF**: breadboard_pin, sb_interface:breadboard_pin, F.Cu at (154.9, 94.0)
- added REF**: breadboard_pin, sb_interface:breadboard_pin, F.Cu at (139.7, 83.8)
- added REF**: breadboard_pin, sb_interface:breadboard_pin, F.Cu at (172.7, 114.3)
- added REF**: breadboard_pin, sb_interface:breadboard_pin, F.Cu at (157.5, 119.4)
- added REF**: breadboard_pin, sb_interface:breadboard_pin, F.Cu at (154.9, 160.0)
- added REF**: breadboard_pin, sb_interface:breadboard_pin, F.Cu at (160.0, 137.2)
- added REF**: breadboard_pin, sb_interface:breadboard_pin, F.Cu at (149.9, 114.3)
- added REF**: breadboard_pin, sb_interface:breadboard_pin, F.Cu at (160.0, 96.5)
- added REF**: breadboard_pin, sb_interface:breadboard_pin, F.Cu at (144.8, 101.6)
- added REF**: breadboard_pin, sb_interface:breadboard_pin, F.Cu at (139.7, 81.3)
- added REF**: breadboard_pin, sb_interface:breadboard_pin, F.Cu at (162.6, 157.5)
- added REF**: breadboard_pin, sb_interface:breadboard_pin, F.Cu at (167.6, 96.5)
- added REF**: breadboard_pin, sb_interface:breadboard_pin, F.Cu at (157.5, 76.2)
- added REF**: breadboard_pin, sb_interface:breadboard_pin, F.Cu at (149.9, 124.5)
- added REF**: breadboard_pin, sb_interface:breadboard_pin, F.Cu at (157.5, 111.8)
- added REF**: breadboard_pin, sb_interface:breadboard_pin, F.Cu at (137.2, 101.6)
- added REF**: breadboard_pin, sb_interface:breadboard_pin, F.Cu at (134.6, 119.4)
- added REF**: breadboard_pin, sb_interface:breadboard_pin, F.Cu at (154.9, 91.4)
- added REF**: breadboard_pin, sb_interface:breadboard_pin, F.Cu at (139.7, 116.8)
- added REF**: breadboard_pin, sb_interface:breadboard_pin, F.Cu at (170.2, 129.5)
- added REF**: breadboard_pin, sb_interface:breadboard_pin, F.Cu at (157.5, 134.6)
- added REF**: breadboard_pin, sb_interface:breadboard_pin, F.Cu at (137.2, 109.2)
- added REF**: breadboard_pin, sb_interface:breadboard_pin, F.Cu at (147.3, 154.9)
- added REF**: breadboard_pin, sb_interface:breadboard_pin, F.Cu at (172.7, 142.2)
- added REF**: breadboard_pin, sb_interface:breadboard_pin, F.Cu at (165.1, 127.0)
- added REF**: breadboard_pin, sb_interface:breadboard_pin, F.Cu at (167.6, 119.4)
- added REF**: breadboard_pin, sb_interface:breadboard_pin, F.Cu at (165.1, 101.6)
- added REF**: breadboard_pin, sb_interface:breadboard_pin, F.Cu at (142.2, 157.5)
- added REF**: breadboard_pin, sb_interface:breadboard_pin, F.Cu at (142.2, 160.0)
- added REF**: breadboard_pin, sb_interface:breadboard_pin, F.Cu at (162.6, 154.9)
- added REF**: breadboard_pin, sb_interface:breadboard_pin, F.Cu at (170.2, 137.2)
- added REF**: breadboard_pin, sb_interface:breadboard_pin, F.Cu at (139.7, 121.9)
- added REF**: breadboard_pin, sb_interface:breadboard_pin, F.Cu at (144.8, 137.2)
- added REF**: breadboard_pin, sb_interface:breadboard_pin, F.Cu at (147.3, 127.0)
- added REF**: breadboard_pin, sb_interface:breadboard_pin, F.Cu at (167.6, 88.9)
- added REF**: breadboard_pin, sb_interface:breadboard_pin, F.Cu at (172.7, 137.2)
- added REF**: breadboard_pin, sb_interface:breadboard_pin, F.Cu at (147.3, 88.9)
- added REF**: breadboard_pin, sb_interface:breadboard_pin, F.Cu at (149.9, 111.8)
- added REF**: breadboard_pin, sb_interface:breadboard_pin, F.Cu at (167.6, 91.4)
- added REF**: breadboard_pin, sb_interface:breadboard_pin, F.Cu at (167.6, 106.7)
- added REF**: breadboard_pin, sb_interface:breadboard_pin, F.Cu at (160.0, 94.0)
- added REF**: breadboard_pin, sb_interface:breadboard_pin, F.Cu at (144.8, 114.3)
- added REF**: breadboard_pin, sb_interface:breadboard_pin, F.Cu at (170.2, 124.5)
- added REF**: breadboard_pin, sb_interface:breadboard_pin, F.Cu at (157.5, 149.9)
- added REF**: breadboard_pin, sb_interface:breadboard_pin, F.Cu at (147.3, 134.6)
- added REF**: breadboard_pin, sb_interface:breadboard_pin, F.Cu at (151.9, 30.5)
- added REF**: breadboard_pin, sb_interface:breadboard_pin, F.Cu at (144.8, 142.2)
- added REF**: breadboard_pin, sb_interface:breadboard_pin, F.Cu at (139.7, 109.2)
- added REF**: breadboard_pin, sb_interface:breadboard_pin, F.Cu at (157.5, 81.3)
- added REF**: breadboard_pin, sb_interface:breadboard_pin, F.Cu at (134.6, 111.8)
- added REF**: breadboard_pin, sb_interface:breadboard_pin, F.Cu at (170.2, 132.1)
- added REF**: breadboard_pin, sb_interface:breadboard_pin, F.Cu at (142.2, 76.2)
- added REF**: breadboard_pin, sb_interface:breadboard_pin, F.Cu at (162.6, 106.7)
- added REF**: breadboard_pin, sb_interface:breadboard_pin, F.Cu at (157.5, 99.1)
- added REF**: breadboard_pin, sb_interface:breadboard_pin, F.Cu at (149.9, 121.9)
- added REF**: breadboard_pin, sb_interface:breadboard_pin, F.Cu at (160.0, 81.3)
- added REF**: breadboard_pin, sb_interface:breadboard_pin, F.Cu at (149.9, 101.6)
- added REF**: breadboard_pin, sb_interface:breadboard_pin, F.Cu at (167.6, 99.1)
- added REF**: breadboard_pin, sb_interface:breadboard_pin, F.Cu at (144.8, 88.9)
- added REF**: breadboard_pin, sb_interface:breadboard_pin, F.Cu at (162.6, 104.1)
- added REF**: breadboard_pin, sb_interface:breadboard_pin, F.Cu at (165.1, 106.7)
- added REF**: breadboard_pin, sb_interface:breadboard_pin, F.Cu at (165.1, 124.5)
- added REF**: breadboard_pin, sb_interface:breadboard_pin, F.Cu at (167.6, 127.0)
- added REF**: breadboard_pin, sb_interface:breadboard_pin, F.Cu at (165.1, 144.8)
- added REF**: breadboard_pin, sb_interface:breadboard_pin, F.Cu at (142.2, 154.9)
- added REF**: breadboard_pin, sb_interface:breadboard_pin, F.Cu at (157.5, 106.7)
- added REF**: breadboard_pin, sb_interface:breadboard_pin, F.Cu at (156.7, 30.5)
- added REF**: breadboard_pin, sb_interface:breadboard_pin, F.Cu at (167.6, 132.1)
- added REF**: breadboard_pin, sb_interface:breadboard_pin, F.Cu at (139.7, 94.0)
- added REF**: breadboard_pin, sb_interface:breadboard_pin, F.Cu at (134.6, 81.3)
- added REF**: breadboard_pin, sb_interface:breadboard_pin, F.Cu at (160.0, 132.1)
- added REF**: breadboard_pin, sb_interface:breadboard_pin, F.Cu at (165.1, 88.9)
- added REF**: breadboard_pin, sb_interface:breadboard_pin, F.Cu at (162.6, 132.1)
- added REF**: breadboard_pin, sb_interface:breadboard_pin, F.Cu at (149.9, 142.2)
- added REF**: breadboard_pin, sb_interface:breadboard_pin, F.Cu at (170.2, 139.7)
- added REF**: breadboard_pin, sb_interface:breadboard_pin, F.Cu at (142.2, 147.3)
- added REF**: breadboard_pin, sb_interface:breadboard_pin, F.Cu at (157.5, 116.8)
- added REF**: breadboard_pin, sb_interface:breadboard_pin, F.Cu at (167.6, 137.2)
- added REF**: breadboard_pin, sb_interface:breadboard_pin, F.Cu at (134.6, 99.1)
- added REF**: breadboard_pin, sb_interface:breadboard_pin, F.Cu at (154.9, 137.2)
- added REF**: breadboard_pin, sb_interface:breadboard_pin, F.Cu at (167.6, 129.5)
- added REF**: breadboard_pin, sb_interface:breadboard_pin, F.Cu at (147.3, 121.9)
- added REF**: breadboard_pin, sb_interface:breadboard_pin, F.Cu at (160.0, 124.5)
- added REF**: breadboard_pin, sb_interface:breadboard_pin, F.Cu at (167.6, 124.5)
- added REF**: breadboard_pin, sb_interface:breadboard_pin, F.Cu at (137.2, 154.9)
- added REF**: breadboard_pin, sb_interface:breadboard_pin, F.Cu at (170.2, 86.4)
- added REF**: breadboard_pin, sb_interface:breadboard_pin, F.Cu at (157.5, 104.1)
- added REF**: breadboard_pin, sb_interface:breadboard_pin, F.Cu at (137.2, 91.4)
- added REF**: breadboard_pin, sb_interface:breadboard_pin, F.Cu at (154.9, 157.5)
- added REF**: breadboard_pin, sb_interface:breadboard_pin, F.Cu at (152.4, 81.3)
- added REF**: breadboard_pin, sb_interface:breadboard_pin, F.Cu at (170.2, 160.0)
- added REF**: breadboard_pin, sb_interface:breadboard_pin, F.Cu at (134.6, 137.2)
- added REF**: breadboard_pin, sb_interface:breadboard_pin, F.Cu at (134.6, 157.5)
- added REF**: breadboard_pin, sb_interface:breadboard_pin, F.Cu at (170.2, 88.9)
- added REF**: breadboard_pin, sb_interface:breadboard_pin, F.Cu at (157.5, 142.2)
- added REF**: breadboard_pin, sb_interface:breadboard_pin, F.Cu at (172.7, 68.6)
- added REF**: breadboard_pin, sb_interface:breadboard_pin, F.Cu at (142.2, 73.7)
- added REF**: breadboard_pin, sb_interface:breadboard_pin, F.Cu at (134.6, 96.5)
- added REF**: breadboard_pin, sb_interface:breadboard_pin, F.Cu at (152.4, 165.1)
- added REF**: breadboard_pin, sb_interface:breadboard_pin, F.Cu at (170.2, 81.3)
- added REF**: breadboard_pin, sb_interface:breadboard_pin, F.Cu at (137.2, 144.8)
- added REF**: breadboard_pin, sb_interface:breadboard_pin, F.Cu at (162.6, 160.0)
- added REF**: breadboard_pin, sb_interface:breadboard_pin, F.Cu at (147.3, 147.3)
- added REF**: breadboard_pin, sb_interface:breadboard_pin, F.Cu at (134.6, 101.6)
- added REF**: breadboard_pin, sb_interface:breadboard_pin, F.Cu at (154.9, 86.4)
- added REF**: breadboard_pin, sb_interface:breadboard_pin, F.Cu at (137.2, 73.7)
- added REF**: breadboard_pin, sb_interface:breadboard_pin, F.Cu at (142.2, 137.2)
- added REF**: breadboard_pin, sb_interface:breadboard_pin, F.Cu at (157.5, 96.5)
- added REF**: breadboard_pin, sb_interface:breadboard_pin, F.Cu at (162.6, 149.9)
- added REF**: breadboard_pin, sb_interface:breadboard_pin, F.Cu at (152.4, 147.3)
- added REF**: breadboard_pin, sb_interface:breadboard_pin, F.Cu at (144.8, 106.7)
- added REF**: breadboard_pin, sb_interface:breadboard_pin, F.Cu at (137.2, 157.5)
- added REF**: breadboard_pin, sb_interface:breadboard_pin, F.Cu at (147.3, 94.0)
- added REF**: breadboard_pin, sb_interface:breadboard_pin, F.Cu at (144.8, 111.8)
- added REF**: breadboard_pin, sb_interface:breadboard_pin, F.Cu at (144.8, 124.5)
- added REF**: breadboard_pin, sb_interface:breadboard_pin, F.Cu at (137.2, 88.9)
- added REF**: breadboard_pin, sb_interface:breadboard_pin, F.Cu at (170.2, 83.8)
- added REF**: breadboard_pin, sb_interface:breadboard_pin, F.Cu at (172.7, 83.8)
- added REF**: breadboard_pin, sb_interface:breadboard_pin, F.Cu at (160.0, 88.9)
- added REF**: breadboard_pin, sb_interface:breadboard_pin, F.Cu at (142.2, 111.8)
- added REF**: breadboard_pin, sb_interface:breadboard_pin, F.Cu at (170.2, 142.2)
- added REF**: breadboard_pin, sb_interface:breadboard_pin, F.Cu at (144.8, 76.2)
- added REF**: breadboard_pin, sb_interface:breadboard_pin, F.Cu at (167.6, 116.8)
- added REF**: breadboard_pin, sb_interface:breadboard_pin, F.Cu at (162.6, 114.3)
- added REF**: breadboard_pin, sb_interface:breadboard_pin, F.Cu at (157.5, 157.5)
- added REF**: breadboard_pin, sb_interface:breadboard_pin, F.Cu at (152.4, 111.8)
- added REF**: breadboard_pin, sb_interface:breadboard_pin, F.Cu at (165.1, 152.4)
- added REF**: breadboard_pin, sb_interface:breadboard_pin, F.Cu at (157.5, 68.6)
- added REF**: breadboard_pin, sb_interface:breadboard_pin, F.Cu at (165.1, 111.8)
- added REF**: breadboard_pin, sb_interface:breadboard_pin, F.Cu at (137.2, 106.7)
- added REF**: breadboard_pin, sb_interface:breadboard_pin, F.Cu at (172.7, 106.7)
- added REF**: breadboard_pin, sb_interface:breadboard_pin, F.Cu at (172.7, 81.3)
- added REF**: breadboard_pin, sb_interface:breadboard_pin, F.Cu at (160.0, 114.3)
- added REF**: breadboard_pin, sb_interface:breadboard_pin, F.Cu at (149.9, 116.8)
- added REF**: breadboard_pin, sb_interface:breadboard_pin, F.Cu at (154.9, 152.4)
- added REF**: breadboard_pin, sb_interface:breadboard_pin, F.Cu at (137.2, 132.1)
- added REF**: breadboard_pin, sb_interface:breadboard_pin, F.Cu at (147.3, 96.5)
- added REF**: breadboard_pin, sb_interface:breadboard_pin, F.Cu at (172.7, 139.7)
- added REF**: breadboard_pin, sb_interface:breadboard_pin, F.Cu at (165.1, 137.2)
- added REF**: breadboard_pin, sb_interface:breadboard_pin, F.Cu at (152.4, 139.7)
- added REF**: breadboard_pin, sb_interface:breadboard_pin, F.Cu at (152.4, 142.2)
- added REF**: breadboard_pin, sb_interface:breadboard_pin, F.Cu at (157.5, 114.3)
- added REF**: breadboard_pin, sb_interface:breadboard_pin, F.Cu at (134.6, 121.9)
- added REF**: breadboard_pin, sb_interface:breadboard_pin, F.Cu at (162.6, 78.7)
- added REF**: breadboard_pin, sb_interface:breadboard_pin, F.Cu at (137.2, 160.0)
- added REF**: breadboard_pin, sb_interface:breadboard_pin, F.Cu at (152.4, 94.0)
- added REF**: breadboard_pin, sb_interface:breadboard_pin, F.Cu at (160.0, 152.4)
- added REF**: breadboard_pin, sb_interface:breadboard_pin, F.Cu at (165.1, 160.0)
- added REF**: breadboard_pin, sb_interface:breadboard_pin, F.Cu at (147.3, 132.1)
- added REF**: breadboard_pin, sb_interface:breadboard_pin, F.Cu at (170.2, 144.8)
- added REF**: breadboard_pin, sb_interface:breadboard_pin, F.Cu at (154.9, 144.8)
- added REF**: breadboard_pin, sb_interface:breadboard_pin, F.Cu at (160.0, 149.9)
- added REF**: breadboard_pin, sb_interface:breadboard_pin, F.Cu at (160.0, 101.6)
- added REF**: breadboard_pin, sb_interface:breadboard_pin, F.Cu at (162.6, 129.5)
- added REF**: breadboard_pin, sb_interface:breadboard_pin, F.Cu at (170.2, 106.7)
- added REF**: breadboard_pin, sb_interface:breadboard_pin, F.Cu at (142.2, 91.4)
- added REF**: breadboard_pin, sb_interface:breadboard_pin, F.Cu at (152.4, 86.4)
- added REF**: breadboard_pin, sb_interface:breadboard_pin, F.Cu at (170.2, 147.3)
- added REF**: breadboard_pin, sb_interface:breadboard_pin, F.Cu at (162.6, 86.4)
- added REF**: breadboard_pin, sb_interface:breadboard_pin, F.Cu at (139.7, 88.9)
- added REF**: breadboard_pin, sb_interface:breadboard_pin, F.Cu at (149.9, 94.0)
- added REF**: breadboard_pin, sb_interface:breadboard_pin, F.Cu at (152.4, 76.2)
- added REF**: breadboard_pin, sb_interface:breadboard_pin, F.Cu at (144.8, 109.2)
- added REF**: breadboard_pin, sb_interface:breadboard_pin, F.Cu at (172.7, 152.4)
- added REF**: breadboard_pin, sb_interface:breadboard_pin, F.Cu at (160.0, 160.0)
- added REF**: breadboard_pin, sb_interface:breadboard_pin, F.Cu at (147.3, 124.5)
- added REF**: breadboard_pin, sb_interface:breadboard_pin, F.Cu at (167.6, 154.9)
- added REF**: breadboard_pin, sb_interface:breadboard_pin, F.Cu at (167.6, 152.4)
- added REF**: breadboard_pin, sb_interface:breadboard_pin, F.Cu at (160.0, 86.4)
- added REF**: breadboard_pin, sb_interface:breadboard_pin, F.Cu at (149.9, 91.4)
- added REF**: breadboard_pin, sb_interface:breadboard_pin, F.Cu at (165.1, 68.6)
- added REF**: breadboard_pin, sb_interface:breadboard_pin, F.Cu at (162.6, 147.3)
- added REF**: breadboard_pin, sb_interface:breadboard_pin, F.Cu at (147.3, 144.8)
- added REF**: breadboard_pin, sb_interface:breadboard_pin, F.Cu at (170.2, 101.6)
- added REF**: breadboard_pin, sb_interface:breadboard_pin, F.Cu at (172.7, 134.6)
- added REF**: breadboard_pin, sb_interface:breadboard_pin, F.Cu at (147.3, 91.4)
- added REF**: breadboard_pin, sb_interface:breadboard_pin, F.Cu at (165.1, 129.5)
- added REF**: breadboard_pin, sb_interface:breadboard_pin, F.Cu at (160.0, 76.2)
- added REF**: breadboard_pin, sb_interface:breadboard_pin, F.Cu at (144.8, 83.8)
- added REF**: breadboard_pin, sb_interface:breadboard_pin, F.Cu at (142.2, 81.3)
- added REF**: breadboard_pin, sb_interface:breadboard_pin, F.Cu at (162.6, 127.0)
- added REF**: breadboard_pin, sb_interface:breadboard_pin, F.Cu at (147.3, 137.2)
- added REF**: breadboard_pin, sb_interface:breadboard_pin, F.Cu at (170.2, 91.4)
- added REF**: breadboard_pin, sb_interface:breadboard_pin, F.Cu at (142.2, 88.9)
- added REF**: breadboard_pin, sb_interface:breadboard_pin, F.Cu at (167.6, 76.2)
- added REF**: breadboard_pin, sb_interface:breadboard_pin, F.Cu at (147.3, 78.7)
- added REF**: breadboard_pin, sb_interface:breadboard_pin, F.Cu at (139.7, 101.6)
- added REF**: breadboard_pin, sb_interface:breadboard_pin, F.Cu at (152.4, 157.5)
- added REF**: breadboard_pin, sb_interface:breadboard_pin, F.Cu at (139.7, 86.4)
- added REF**: breadboard_pin, sb_interface:breadboard_pin, F.Cu at (165.1, 96.5)
- added REF**: breadboard_pin, sb_interface:breadboard_pin, F.Cu at (142.2, 127.0)
- added REF**: breadboard_pin, sb_interface:breadboard_pin, F.Cu at (160.0, 127.0)
- added REF**: breadboard_pin, sb_interface:breadboard_pin, F.Cu at (170.2, 154.9)
- added REF**: breadboard_pin, sb_interface:breadboard_pin, F.Cu at (152.4, 96.5)
- added REF**: breadboard_pin, sb_interface:breadboard_pin, F.Cu at (152.4, 116.8)
- added REF**: breadboard_pin, sb_interface:breadboard_pin, F.Cu at (144.8, 116.8)
- added REF**: breadboard_pin, sb_interface:breadboard_pin, F.Cu at (170.2, 134.6)
- added REF**: breadboard_pin, sb_interface:breadboard_pin, F.Cu at (149.9, 76.2)
- added REF**: breadboard_pin, sb_interface:breadboard_pin, F.Cu at (139.7, 132.1)
- added REF**: breadboard_pin, sb_interface:breadboard_pin, F.Cu at (170.2, 78.7)
- added REF**: breadboard_pin, sb_interface:breadboard_pin, F.Cu at (154.9, 96.5)
- added REF**: breadboard_pin, sb_interface:breadboard_pin, F.Cu at (139.7, 152.4)
- added REF**: breadboard_pin, sb_interface:breadboard_pin, F.Cu at (172.7, 94.0)
- added REF**: breadboard_pin, sb_interface:breadboard_pin, F.Cu at (152.4, 132.1)
- added REF**: breadboard_pin, sb_interface:breadboard_pin, F.Cu at (152.4, 73.7)
- added REF**: breadboard_pin, sb_interface:breadboard_pin, F.Cu at (134.6, 114.3)
- added REF**: breadboard_pin, sb_interface:breadboard_pin, F.Cu at (160.0, 157.5)
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Routing:
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- removed copper zone on B.Cu, net +3.3V
Other:
- board size 147.4 x 208.5 mm -> 146.1 x 208.5 mm
- board text added: "+12V"
- board text added: "+3.3V"
- board text added: "A"
- board text added: "B"
- board text added: "GND"
- board text added: "GPA0"
- board text added: "GPA1"
- board text added: "GPA2"
- board text added: "GPA3"
- board text added: "GPA4"
- board text added: "GPA5"
- board text added: "GPA6"
- board text added: "INTA_1"
- board text added: "INTA_2"
- board text added: "INTB_1"
- board text added: "INTB_2"
- board text added: "RST"
- board text added: "SCL"
- board text added: "SDA"
